File: MiniAdder.kicad_pcb (KiCad board)
At the start: 2 copper layers, 35.6 x 50.8 mm, 39 parts, among them J1 SMA, J2 SMA, J3 Conn_01x03_Pin, J4 Conn_01x03_Pin, J5 SMA, J6 SMA, SW1 SS12D07VG2_087, U1 GS8634, U2 ME2188A50XG

Commit message: Update version imformation
Other:
- board text added: "MiniAdder Rev1.1 Designed by CyberMomo"
